Commit message: Modified kuka arm xacro to create a stand alone urdf

File: iai_kuka_lwr4_description/urdf/kuka_lwr_arm.urdf.xacro (robot description, xacro)
@@ -1,22 +1,26 @@
 <?xml version="1.0"?>
-<robot xmlns:sensor="http://playerstage.sourceforge.net/gazebo/xmlschema/#sensor"
+<robot xmlns:xacro="http://www.ros.org/wiki/xacro" name="kuka_lwr_arm"
+       xmlns:sensor="http://playerstage.sourceforge.net/gazebo/xmlschema/#sensor"
        xmlns:controller="http://playerstage.sourceforge.net/gazebo/xmlschema/#controller"
        xmlns:interface="http://playerstage.sourceforge.net/gazebo/xmlschema/#interface">
-  <include filename="$(find iai_kuka_lwr4_description)/defs/util_defs.xml"/>
-  <property name="arm_elem_base_mass" value="2.0"/>
-  <property name="arm_elem_link_mass" value="2.0"/>
-  <property name="arm_elem_ball_link_mass" value="2.0"/>
-  <property name="arm_elem_end_link_mass" value="2.0"/>
-  <property name="arm_elem_flange_link_mass" value="0.5"/>
-  <property name="safety_controller_k_pos" value="100" />
-  <property name="safety_controller_k_vel" value="2" />
-  <property name="joint_damping" value="0.1" />
-  <property name="arm_velocity_scale_factor" value="1"/>
-  <macro name="kuka_lwr_arm" params="parent name *origin">
+  <xacro:include filename="$(find iai_kuka_lwr4_description)/defs/util_defs.xml"/>
+  <xacro:property name="arm_elem_base_mass" value="2.0"/>
+  <xacro:property name="arm_elem_link_mass" value="2.0"/>
+  <xacro:property name="arm_elem_ball_link_mass" value="2.0"/>
+  <xacro:property name="arm_elem_end_link_mass" value="2.0"/>
+  <xacro:property name="arm_elem_flange_link_mass" value="0.5"/>
+  <xacro:property name="safety_controller_k_pos" value="100" />
+  <xacro:property name="safety_controller_k_vel" value="2" />
+  <xacro:property name="joint_damping" value="0.1" />
+  <xacro:property name="arm_velocity_scale_factor" value="1"/>
+  <xacro:macro name="kuka_lwr_arm" params="parent name *origin">
     <joint name="${parent}_${name}_arm_base_joint" type="fixed">
-      <insert_block name="origin"/>
+      <xacro:insert_block name="origin"/>
       <parent link="${parent}"/>
       <child link="calib_${name}_arm_base_link"/>
     </joint>
+    <xacro:kuka_lwr_arm_unconnected name="${name}" />
+  </xacro:macro>
+  <xacro:macro name="kuka_lwr_arm_unconnected" params="name">
     <link name="calib_${name}_arm_base_link">
       <inertial>
@@ -383,4 +387,5 @@
     </joint>
     <link name="${name}_arm_hand_link" / -->
-  </macro>
+  </xacro:macro>
+  <xacro:kuka_lwr_arm_unconnected name="kuka_arm" />
 </robot>
